Commit message: Modify link Inertial parameters

File: sciurus17_description/urdf/sciurus17.urdf (robot description, URDF)
Before this commit: robot sciurus17, 26 links, 25 joints
Links:
- link base_link: mass 0.387313 -> 1722.937e-03
- link body_link: mass 0.387313 -> 1482.929e-03
- link camera_link: mass 0.1 -> None
- link chest_camera_link: mass 0.1 -> None
- link l_handA_link: mass 0.119807 -> 15.8e-03
- link l_handB_link: mass 0.119807 -> 13.9e-03
- link l_link1: mass 0.340878 -> 258.0e-03
- link l_link2: mass 0.230634 -> 134.0e-03
- link l_link3: mass 0.192709 -> 443.0e-03
- link l_link4: mass 0.130549 -> 238.0e-03
- link l_link5: mass 0.119807 -> 224.0e-03
- link l_link6: mass 0.119807 -> 140.0e-03
- link l_link7: mass 0.119807 -> 121.0e-03
- link neck_pitch_link: mass 0.235377 -> 312.172e-03
- link neck_yaw_link: mass 0.120005 -> 168.0e-03
- link r_handA_link: mass 0.119807 -> 15.8e-03
- link r_handB_link: mass 0.119807 -> 13.9e-03
- link r_link1: mass 0.340878 -> 258.0e-03
- link r_link2: mass 0.230634 -> 134.0e-03
- link r_link3: mass 0.192709 -> 443.0e-03
- link r_link4: mass 0.130549 -> 238.0e-03
- link r_link5: mass 0.119807 -> 224.0e-03
- link r_link6: mass 0.119807 -> 140.0e-03; geometry collision mesh filename=package://sciurus17_description/meshes/collision/R_Link6.stl scale=1.0 1.0 1.0; visual mesh filename=package://sciurus17_description/meshes/visual/R_Link6.stl scale=1.0 1.0 1.0
- link r_link7: mass 0.119807 -> 121.0e-03
