Commit message: Add damping & friction values to xacro file

File: sciurus17_description/urdf/sciurus17_body.xacro (robot description, xacro)
@@ -39,4 +39,5 @@
         velocity="${waist_yaw_velocity_limit}"/>
       <axis xyz="0 0 1"/>
+      <dynamics damping="1.0e-6" friction="0.8"/>
     </joint>
     <link name="body_link">

File: sciurus17_description/urdf/sciurus17_gazebo.xacro (robot description, xacro)
@@ -17,46 +17,85 @@
     </transmission>
   </xacro:macro>
-  <gazebo reference="camera_link">
-      <sensor type="depth" name="openni_camera_camera">
-          <always_on>1</always_on>
-          <visualize>true</visualize>
-          <camera>
-              <horizontal_fov>1.047</horizontal_fov>
-              <image>
-                  <width>640</width>
-                  <height>480</height>
-                  <format>R8G8B8</format>
-              </image>
-              <depth_camera>
-              </depth_camera>
-              <clip>
-                  <near>0.1</near>
-                  <far>100</far>
-              </clip>
-          </camera>
-          <plugin name="camera_controller" filename="libgazebo_ros_openni_kinect.so">
-              <robotNamespace>sciurus17</robotNamespace>
-              <alwaysOn>true</alwaysOn>
-                  <updateRate>10.0</updateRate>
-                  <cameraName>camera</cameraName>
-                  <frameName>openni_camera_link</frameName>
-              <imageTopicName>rgb/image_raw</imageTopicName>
-              <depthImageTopicName>depth/image_raw</depthImageTopicName>
-              <pointCloudTopicName>depth/points</pointCloudTopicName>
-              <cameraInfoTopicName>rgb/camera_info</cameraInfoTopicName>
-              <depthImageCameraInfoTopicName>depth/camera_info</depthImageCameraInfoTopicName>
-              <pointCloudCutoff>0.4</pointCloudCutoff>
-                  <hackBaseline>0.07</hackBaseline>
-                  <distortionK1>0.0</distortionK1>
-                  <distortionK2>0.0</distortionK2>
-                  <distortionK3>0.0</distortionK3>
-                  <distortionT1>0.0</distortionT1>
-                  <distortionT2>0.0</distortionT2>
-              <CxPrime>0.0</CxPrime>
-              <Cx>0.0</Cx>
-              <Cy>0.0</Cy>
-              <focalLength>0.0</focalLength>
-          </plugin>
-      </sensor>
+  <gazebo reference="body_link">
+    <sensor name='camera1' type='camera'>
+      <update_rate>30</update_rate>
+      <camera name='head'>
+        <horizontal_fov>1.39626</horizontal_fov>
+        <image>
+          <width>1280</width>
+          <height>800</height>
+          <format>R8G8B8</format>
+        </image>
+        <clip>
+          <near>0.02</near>
+          <far>300</far>
+        </clip>
+        <noise>
+          <type>gaussian</type>
+          <mean>0</mean>
+          <stddev>0.007</stddev>
+        </noise>
+      </camera>
+      <plugin name='camera_controller' filename='libgazebo_ros_camera.so'>
+        <alwaysOn>true</alwaysOn>
+        <updateRate>0.0</updateRate>
+        <cameraName>sciurus17/chest_camera_node</cameraName>
+        <imageTopicName>image</imageTopicName>
+        <cameraInfoTopicName>camera_info</cameraInfoTopicName>
+        <frameName>chest_camera_link</frameName>
+        <hackBaseline>0.07</hackBaseline>
+        <distortionK1>0.0</distortionK1>
+        <distortionK2>0.0</distortionK2>
+        <distortionK3>0.0</distortionK3>
+        <distortionT1>0.0</distortionT1>
+        <distortionT2>0.0</distortionT2>
+      </plugin>
+      <pose frame=''>0.114576 0 0.217659 0 0.5236 0</pose>
+    </sensor>
+  </gazebo>
+  <gazebo reference="neck_pitch_link">
+    <sensor name='openni_camera_camera' type='depth'>
+      <always_on>1</always_on>
+      <visualize>1</visualize>
+      <camera name='__default__'>
+        <horizontal_fov>1.047</horizontal_fov>
+        <image>
+          <width>640</width>
+          <height>480</height>
+          <format>R8G8B8</format>
+        </image>
+        <depth_camera>
+          <output>depths</output>
+        </depth_camera>
+        <clip>
+          <near>0.1</near>
+          <far>100</far>
+        </clip>
+      </camera>
+      <plugin name='camera_controller' filename='libgazebo_ros_openni_kinect.so'>
+        <robotNamespace>sciurus17</robotNamespace>
+        <alwaysOn>true</alwaysOn>
+        <updateRate>10.0</updateRate>
+        <cameraName>camera</cameraName>
+        <frameName>openni_camera_link</frameName>
+        <imageTopicName>color/image_raw</imageTopicName>
+        <depthImageTopicName>depth/image_raw</depthImageTopicName>
+        <pointCloudTopicName>depth/points</pointCloudTopicName>
+        <cameraInfoTopicName>color/camera_info</cameraInfoTopicName>
+        <depthImageCameraInfoTopicName>depth/camera_info</depthImageCameraInfoTopicName>
+        <pointCloudCutoff>0.4</pointCloudCutoff>
+        <hackBaseline>0.07</hackBaseline>
+        <distortionK1>0.0</distortionK1>
+        <distortionK2>0.0</distortionK2>
+        <distortionK3>0.0</distortionK3>
+        <distortionT1>0.0</distortionT1>
+        <distortionT2>0.0</distortionT2>
+        <CxPrime>0.0</CxPrime>
+        <Cx>0.0</Cx>
+        <Cy>0.0</Cy>
+        <focalLength>0.0</focalLength>
+      </plugin>
+      <pose frame=''>0.081785 0.03522 0.091 0 -0 0</pose>
+    </sensor>
   </gazebo>
   <gazebo>

File: sciurus17_description/urdf/sciurus17_head.xacro (robot description, xacro)
@@ -21,4 +21,5 @@
         velocity="${neck_joints_velocity_limit}"/>
       <axis xyz="0 0 1"/>
+      <dynamics damping="1.0e-6" friction="0.8"/>
     </joint>
     <link name="neck_yaw_link">
@@ -50,4 +51,5 @@
         velocity="${neck_joints_velocity_limit}"/>
       <axis xyz="0 -1 0"/>
+      <dynamics damping="1.0e-6" friction="0.8"/>
     </joint>
     <link name="neck_pitch_link">

File: sciurus17_description/urdf/sciurus17_left_arm.xacro (robot description, xacro)
@@ -30,4 +30,5 @@
         velocity="${arm_joints_velocity_limit}"/>
       <axis xyz="0 1 0"/>
+      <dynamics damping="1.0e-6" friction="0.8"/>
     </joint>
     <link name="l_link1">
@@ -61,4 +62,5 @@
         velocity="${arm_joints_velocity_limit}"/>
       <axis xyz="-1 0 0"/>
+      <dynamics damping="1.0e-6" friction="0.8"/>
     </joint>
     <link name="l_link2">
@@ -92,4 +94,5 @@
         velocity="${arm_joints_velocity_limit}"/>
       <axis xyz="0 1 0"/>
+      <dynamics damping="1.0e-6" friction="0.8"/>
     </joint>
     <link name="l_link3">
@@ -123,4 +126,5 @@
         velocity="${arm_joints_velocity_limit}"/>
       <axis xyz="0 0 1"/>
+      <dynamics damping="1.0e-6" friction="0.8"/>
     </joint>
     <link name="l_link4">
@@ -154,4 +158,5 @@
         velocity="${arm_joints_velocity_limit}"/>
       <axis xyz="0 1 0"/>
+      <dynamics damping="1.0e-6" friction="0.8"/>
     </joint>
     <link name="l_link5">
@@ -217,4 +222,5 @@
         velocity="${arm_joints_velocity_limit}"/>
       <axis xyz="0 0 1"/>
+      <dynamics damping="1.0e-6" friction="0.8"/>
     </joint>
     <link name="l_link6">
@@ -248,4 +254,5 @@
         velocity="${arm_joints_velocity_limit}"/>
       <axis xyz="0 1 0"/>
+      <dynamics damping="1.0e-6" friction="0.8"/>
     </joint>
   </xacro:macro>

File: sciurus17_description/urdf/sciurus17_left_hand.xacro (robot description, xacro)
@@ -38,4 +38,5 @@
         velocity="${hand_joints_velocity_limit}"/>
       <axis xyz="0 0 1"/>
+      <dynamics damping="1.0e-6" friction="0.8"/>
     </joint>
     <link name="l_handA_link">
@@ -70,4 +71,5 @@
       <axis xyz="0 0 1"/>
       <mimic joint="l_hand_joint" multiplier="-1" offset="0"/>
+      <dynamics damping="1.0e-6" friction="0.8"/>
     </joint>
     <link name="l_handB_link">

File: sciurus17_description/urdf/sciurus17_right_arm.xacro (robot description, xacro)
@@ -30,4 +30,5 @@
         velocity="${arm_joints_velocity_limit}"/>
       <axis xyz="0 -1 0"/>
+      <dynamics damping="1.0e-6" friction="0.8"/>
     </joint>
     <link name="r_link1">
@@ -61,4 +62,5 @@
         velocity="${arm_joints_velocity_limit}"/>
       <axis xyz="-1 0 0"/>
+      <dynamics damping="1.0e-6" friction="0.8"/>
     </joint>
     <link name="r_link2">
@@ -92,4 +94,5 @@
         velocity="${arm_joints_velocity_limit}"/>
       <axis xyz="0 -1 0"/>
+      <dynamics damping="1.0e-6" friction="0.8"/>
     </joint>
     <link name="r_link3">
@@ -123,4 +126,5 @@
         velocity="${arm_joints_velocity_limit}"/>
       <axis xyz="0 0 1"/>
+      <dynamics damping="1.0e-6" friction="0.8"/>
     </joint>
     <link name="r_link4">
@@ -154,4 +158,5 @@
         velocity="${arm_joints_velocity_limit}"/>
       <axis xyz="0 -1 0"/>
+      <dynamics damping="1.0e-6" friction="0.8"/>
     </joint>
     <link name="r_link5">
@@ -217,4 +222,5 @@
         velocity="${arm_joints_velocity_limit}"/>
       <axis xyz="0 0 1"/>
+      <dynamics damping="1.0e-6" friction="0.8"/>
     </joint>
     <link name="r_link6">
@@ -248,4 +254,5 @@
         velocity="${arm_joints_velocity_limit}"/>
       <axis xyz="0 -1 0"/>
+      <dynamics damping="1.0e-6" friction="0.8"/>
     </joint>
   </xacro:macro>

File: sciurus17_description/urdf/sciurus17_right_hand.xacro (robot description, xacro)
@@ -38,4 +38,5 @@
         velocity="${hand_joints_velocity_limit}"/>
       <axis xyz="0 0 1"/>
+      <dynamics damping="1.0e-6" friction="0.8"/>
     </joint>
     <link name="r_handA_link">
@@ -71,4 +72,5 @@
       <axis xyz="0 0 1"/>
       <mimic joint="r_hand_joint" multiplier="-1" offset="0"/>
+      <dynamics damping="1.0e-6" friction="0.8"/>
     </joint>
     <link name="r_handB_link">

Commit message: Add material configurations to xacro files

File: sciurus17_description/urdf/sciurus17_body.xacro (robot description, xacro)
@@ -80,4 +80,13 @@
       </collision>
     </link>
+    <gazebo reference="base_link">
+      <material>Gazebo/White</material>
+    </gazebo>
+    <gazebo reference="body_link">
+      <material>Gazebo/White</material>
+    </gazebo>
+    <gazebo reference="chest_camera_link">
+      <material>Gazebo/Black</material>
+    </gazebo>
   </xacro:macro>
 </robot>

File: sciurus17_description/urdf/sciurus17_head.xacro (robot description, xacro)
@@ -93,4 +93,13 @@
       </collision>
     </link>
+    <gazebo reference="neck_yaw_link">
+      <material>Gazebo/White</material>
+    </gazebo>
+    <gazebo reference="neck_pitch_link">
+      <material>Gazebo/White</material>
+    </gazebo>
+    <gazebo reference="camera_link">
+      <material>Gazebo/Black</material>
+    </gazebo>
   </xacro:macro>
 </robot>

File: sciurus17_description/urdf/sciurus17_left_arm.xacro (robot description, xacro)
@@ -256,4 +256,22 @@
       <dynamics damping="1.0e-6" friction="0.8"/>
     </joint>
+    <gazebo reference="l_link1">
+      <material>Gazebo/White</material>
+    </gazebo>
+    <gazebo reference="l_link2">
+      <material>Gazebo/White</material>
+    </gazebo>
+    <gazebo reference="l_link3">
+      <material>Gazebo/White</material>
+    </gazebo>
+    <gazebo reference="l_link4">
+      <material>Gazebo/White</material>
+    </gazebo>
+    <gazebo reference="l_link5">
+      <material>Gazebo/White</material>
+    </gazebo>
+    <gazebo reference="l_link6">
+      <material>Gazebo/White</material>
+    </gazebo>
   </xacro:macro>
 </robot>

File: sciurus17_description/urdf/sciurus17_left_hand.xacro (robot description, xacro)
@@ -93,4 +93,13 @@
       </inertial>
     </link>
+    <gazebo reference="l_link7">
+      <material>Gazebo/Red</material>
+    </gazebo>
+    <gazebo reference="l_handA_link">
+      <material>Gazebo/Red</material>
+    </gazebo>
+    <gazebo reference="l_handB_link">
+      <material>Gazebo/Red</material>
+    </gazebo>
   </xacro:macro>
 </robot>

File: sciurus17_description/urdf/sciurus17_right_arm.xacro (robot description, xacro)
@@ -256,4 +256,22 @@
       <dynamics damping="1.0e-6" friction="0.8"/>
     </joint>
+    <gazebo reference="r_link1">
+      <material>Gazebo/White</material>
+    </gazebo>
+    <gazebo reference="r_link2">
+      <material>Gazebo/White</material>
+    </gazebo>
+    <gazebo reference="r_link3">
+      <material>Gazebo/White</material>
+    </gazebo>
+    <gazebo reference="r_link4">
+      <material>Gazebo/White</material>
+    </gazebo>
+    <gazebo reference="r_link5">
+      <material>Gazebo/White</material>
+    </gazebo>
+    <gazebo reference="r_link6">
+      <material>Gazebo/White</material>
+    </gazebo>
   </xacro:macro>
 </robot>

File: sciurus17_description/urdf/sciurus17_right_hand.xacro (robot description, xacro)
@@ -95,4 +95,13 @@
       </inertial>
     </link>
+    <gazebo reference="r_link7">
+      <material>Gazebo/Red</material>
+    </gazebo>
+    <gazebo reference="r_handA_link">
+      <material>Gazebo/Red</material>
+    </gazebo>
+    <gazebo reference="r_handB_link">
+      <material>Gazebo/Red</material>
+    </gazebo>
   </xacro:macro>
 </robot>
