Commit message: Fix head_camera_joint of URDF

File: sciurus17_description/urdf/sciurus17_head.xacro (robot description, xacro)
@@ -76,5 +76,5 @@
       <parent link="neck_pitch_link" />
       <child link="camera_link" />
-      <origin xyz="0.081785 0.03522 0.091" rpy="0 0 0"/>
+      <origin xyz="0.081785 0.020 0.091" rpy="0 0 0"/>
     </joint>
     <link name="camera_link">
