Commit message: Fix gripper mimic joint angles

File: sciurus17_description/urdf/sciurus17_left_hand.xacro (robot description, xacro)
@@ -70,5 +70,5 @@
         velocity="${hand_joints_velocity_limit}"/>
       <axis xyz="0 0 -1"/>
-      <mimic joint="l_hand_joint" multiplier="-1" offset="0"/>
+      <mimic joint="l_hand_joint" multiplier="1" offset="0"/>
       <dynamics damping="1.0e-6" friction="0.8"/>
     </joint>

File: sciurus17_description/urdf/sciurus17_right_hand.xacro (robot description, xacro)
@@ -71,5 +71,5 @@
         velocity="${hand_joints_velocity_limit}"/>
       <axis xyz="0 0 -1"/>
-      <mimic joint="r_hand_joint" multiplier="-1" offset="0"/>
+      <mimic joint="r_hand_joint" multiplier="1" offset="0"/>
       <dynamics damping="1.0e-6" friction="0.8"/>
     </joint>
