Commit message: Add mimic_joint_plugin for sciurus17_gazebo

File: sciurus17_description/urdf/sciurus17_gazebo.xacro (robot description, xacro)
@@ -5,5 +5,5 @@
     <transmission name="${joint_name}_trans">
       <provideFeedback>true</provideFeedback>
-      <implicitSpringDamper>1</implicitSpringDamper>
+      <implicitSpringDamper>0</implicitSpringDamper>
       <motorTorqueConstant>0.418</motorTorqueConstant>
       <type>transmission_interface/SimpleTransmission</type>
@@ -115,4 +115,14 @@
       <legacyModeNS>true</legacyModeNS>
     </plugin>
+    <plugin name="r_hand_mimic_joint_plugin" filename="libroboticsgroup_gazebo_mimic_joint_plugin.so">
+      <joint>r_hand_joint</joint>
+      <mimicJoint>r_hand_mimic_joint</mimicJoint>
+      <multiplier>1.0</multiplier>
+    </plugin>
+    <plugin name="l_hand_mimic_joint_plugin" filename="libroboticsgroup_gazebo_mimic_joint_plugin.so">
+      <joint>l_hand_joint</joint>
+      <mimicJoint>l_hand_mimic_joint</mimicJoint>
+      <multiplier>1.0</multiplier>
+    </plugin>
   </gazebo>
 </robot>

File: sciurus17_description/urdf/sciurus17_left_hand.xacro (robot description, xacro)
@@ -69,5 +69,5 @@
         effort="${hand_joints_effort_limit}"
         velocity="${hand_joints_velocity_limit}"/>
-      <axis xyz="0 0 1"/>
+      <axis xyz="0 0 -1"/>
       <mimic joint="l_hand_joint" multiplier="-1" offset="0"/>
       <dynamics damping="1.0e-6" friction="0.8"/>

File: sciurus17_description/urdf/sciurus17_right_hand.xacro (robot description, xacro)
@@ -70,5 +70,5 @@
         effort="${hand_joints_effort_limit}"
         velocity="${hand_joints_velocity_limit}"/>
-      <axis xyz="0 0 1"/>
+      <axis xyz="0 0 -1"/>
       <mimic joint="r_hand_joint" multiplier="-1" offset="0"/>
       <dynamics damping="1.0e-6" friction="0.8"/>

Commit message: Fix frameName and color format, add camera_color_optical_frame link

File: sciurus17_description/urdf/sciurus17_gazebo.xacro (robot description, xacro)
@@ -63,5 +63,5 @@
           <width>640</width>
           <height>480</height>
-          <format>R8G8B8</format>
+          <format>B8G8R8</format>
         </image>
         <depth_camera>
@@ -78,5 +78,5 @@
         <updateRate>10.0</updateRate>
         <cameraName>camera</cameraName>
-        <frameName>openni_camera_link</frameName>
+        <frameName>/camera_color_optical_frame</frameName>
         <imageTopicName>color/image_raw</imageTopicName>
         <depthImageTopicName>depth/image_raw</depthImageTopicName>
@@ -99,4 +99,10 @@
     </sensor>
   </gazebo>
+  <joint name="camera_color_optical_joint" type="fixed">
+    <origin xyz="0 0.015 0" rpy="-1.5708 0 -1.5708"/>
+    <parent link="camera_link"/>
+    <child link="camera_color_optical_frame"/>
+  </joint>
+  <link name="camera_color_optical_frame"/>
   <gazebo>
     <plugin name='gazebo_ros_control1' filename='libgazebo_ros_control.so'>

Commit message: Add camera_depth_optical_joint to xacro file

File: sciurus17_description/urdf/sciurus17_gazebo.xacro (robot description, xacro)
@@ -105,4 +105,10 @@
   </joint>
   <link name="camera_color_optical_frame"/>
+  <joint name="camera_depth_optical_joint" type="fixed">
+    <origin xyz="0 0.015 0" rpy="-1.5708 0 -1.5708"/>
+    <parent link="camera_link"/>
+    <child link="camera_depth_optical_frame"/>
+  </joint>
+  <link name="camera_depth_optical_frame"/>
   <gazebo>
     <plugin name='gazebo_ros_control1' filename='libgazebo_ros_control.so'>
