Commit message: Fix arm model scale

File: sciurus17_description/urdf/sciurus17_left_arm.xacro (robot description, xacro)
@@ -68,5 +68,5 @@
         <origin rpy="0 -1.5708 0" xyz="0.0 0.0 0.0"/>
         <geometry>
-          <mesh filename="package://sciurus17_description/meshes/visual/L_Link2.stl" scale="1.0 1.0 -1.0"/>
+          <mesh filename="package://sciurus17_description/meshes/visual/L_Link2.stl" scale="-1.0 1.0 -1.0"/>
         </geometry>
         <material name="${arm_color}"/>
@@ -75,5 +75,5 @@
         <origin rpy="0 -1.5708 0" xyz="0.0 0.0 0.0"/>
         <geometry>
-          <mesh filename="package://sciurus17_description/meshes/collision/L_Link2.stl" scale="1.0 1.0 -1.0"/>
+          <mesh filename="package://sciurus17_description/meshes/collision/L_Link2.stl" scale="-1.0 1.0 -1.0"/>
         </geometry>
       </collision>

File: sciurus17_description/urdf/sciurus17_right_arm.xacro (robot description, xacro)
@@ -68,5 +68,5 @@
         <origin rpy="0 1.5708 0" xyz="0.0 0.0 0.0"/>
         <geometry>
-          <mesh filename="package://sciurus17_description/meshes/visual/R_Link2.stl" scale="-1.0 1.0 1.0"/>
+          <mesh filename="package://sciurus17_description/meshes/visual/R_Link2.stl" scale="1.0 1.0 1.0"/>
         </geometry>
         <material name="${arm_color}"/>
@@ -75,5 +75,5 @@
         <origin rpy="0 1.5708 0" xyz="0.0 0.0 0.0"/>
         <geometry>
-          <mesh filename="package://sciurus17_description/meshes/collision/R_Link2.stl" scale="-1.0 1.0 1.0"/>
+          <mesh filename="package://sciurus17_description/meshes/collision/R_Link2.stl" scale="1.0 1.0 1.0"/>
         </geometry>
       </collision>

Commit message: Add collision model to armarker link

File: sciurus17_description/urdf/sciurus17_left_arm.xacro (robot description, xacro)
@@ -211,4 +211,10 @@
         <material name="${arm_color}"/>
       </visual>
+      <collision>
+        <origin rpy="0 0 0" xyz="0.0 0.0 0.0"/>
+        <geometry>
+          <cylinder length="0.001" radius="0.001"/>
+        </geometry>
+      </collision>
     </link>
     <joint name="l_arm_joint6" type="revolute">

File: sciurus17_description/urdf/sciurus17_right_arm.xacro (robot description, xacro)
@@ -211,4 +211,10 @@
         <material name="${arm_color}"/>
       </visual>
+      <collision>
+        <origin rpy="0 0 0" xyz="0.0 0.0 0.0"/>
+        <geometry>
+          <cylinder length="0.001" radius="0.001"/>
+        </geometry>
+      </collision>
     </link>
     <joint name="r_arm_joint6" type="revolute">
