Commit message: sciuru17_gazebo launches simulation with xacro file. (without .sdf file)

File: sciurus17_description/urdf/sciurus17.urdf.xacro (robot description, xacro)
@@ -16,23 +16,40 @@
   <xacro:property name="VELOCITY_LIMIT" value="5.969211435"/>
   <xacro:arg name="use_gazebo_simulation" default="false" />
+  <xacro:arg name="load_trans1" default="false" />
+  <xacro:arg name="load_trans2" default="false" />
+  <xacro:arg name="load_trans3" default="false" />
   <xacro:if value="$(arg use_gazebo_simulation)">
     <xacro:include filename="$(find sciurus17_description)/urdf/sciurus17_gazebo.xacro"/>
-    <xacro:default_transmission joint_name="waist_yaw_joint"/>
-    <xacro:default_transmission joint_name="neck_yaw_joint"/>
-    <xacro:default_transmission joint_name="neck_pitch_joint"/>
-    <xacro:default_transmission joint_name="r_arm_joint1"/>
-    <xacro:default_transmission joint_name="r_arm_joint2"/>
-    <xacro:default_transmission joint_name="r_arm_joint3"/>
-    <xacro:default_transmission joint_name="r_arm_joint4"/>
-    <xacro:default_transmission joint_name="r_arm_joint5"/>
-    <xacro:default_transmission joint_name="r_arm_joint6"/>
-    <xacro:default_transmission joint_name="r_arm_joint7"/>
-    <xacro:default_transmission joint_name="l_arm_joint1"/>
-    <xacro:default_transmission joint_name="l_arm_joint2"/>
-    <xacro:default_transmission joint_name="l_arm_joint3"/>
-    <xacro:default_transmission joint_name="l_arm_joint4"/>
-    <xacro:default_transmission joint_name="l_arm_joint5"/>
-    <xacro:default_transmission joint_name="l_arm_joint6"/>
-    <xacro:default_transmission joint_name="l_arm_joint7"/>
+    <xacro:if value="$(arg load_trans1)">
+      <xacro:default_transmission joint_name="r_arm_joint1"/>
+      <xacro:default_transmission joint_name="r_arm_joint2"/>
+      <xacro:default_transmission joint_name="r_arm_joint3"/>
+      <xacro:default_transmission joint_name="r_arm_joint4"/>
+      <xacro:default_transmission joint_name="r_arm_joint5"/>
+      <xacro:default_transmission joint_name="r_arm_joint6"/>
+      <xacro:default_transmission joint_name="r_arm_joint7"/>
+      <xacro:default_transmission joint_name="r_hand_joint"/>
+    </xacro:if>
+    <xacro:if value="$(arg load_trans2)">
+      <xacro:default_transmission joint_name="l_arm_joint1"/>
+      <xacro:default_transmission joint_name="l_arm_joint2"/>
+      <xacro:default_transmission joint_name="l_arm_joint3"/>
+      <xacro:default_transmission joint_name="l_arm_joint4"/>
+      <xacro:default_transmission joint_name="l_arm_joint5"/>
+      <xacro:default_transmission joint_name="l_arm_joint6"/>
+      <xacro:default_transmission joint_name="l_arm_joint7"/>
+      <xacro:default_transmission joint_name="l_hand_joint"/>
+    </xacro:if>
+    <xacro:if value="$(arg load_trans3)">
+      <xacro:default_transmission joint_name="waist_yaw_joint"/>
+      <xacro:default_transmission joint_name="neck_yaw_joint"/>
+      <xacro:default_transmission joint_name="neck_pitch_joint"/>
+    </xacro:if>
+    <!-- Used for fixing robot 'base_link'  to Gazebo 'world' -->
+    <link name="world"/>
+    <joint name="base_link_to_world_joint" type="fixed">
+      <parent link="world"/>
+      <child link="base_link"/>
+    </joint>
   </xacro:if>
   <sciurus17_body

File: sciurus17_description/urdf/sciurus17_gazebo.xacro (robot description, xacro)
@@ -60,3 +60,20 @@
       </sensor>
   </gazebo>
+  <gazebo>
+    <plugin name='gazebo_ros_control1' filename='libgazebo_ros_control.so'>
+      <robotNamespace>/sciurus17/controller1</robotNamespace>
+      <robotSimType>gazebo_ros_control/DefaultRobotHWSim</robotSimType>
+      <legacyModeNS>true</legacyModeNS>
+    </plugin>
+    <plugin name='gazebo_ros_control2' filename='libgazebo_ros_control.so'>
+      <robotNamespace>/sciurus17/controller2</robotNamespace>
+      <robotSimType>gazebo_ros_control/DefaultRobotHWSim</robotSimType>
+      <legacyModeNS>true</legacyModeNS>
+    </plugin>
+    <plugin name='gazebo_ros_control3' filename='libgazebo_ros_control.so'>
+      <robotNamespace>/sciurus17/controller3</robotNamespace>
+      <robotSimType>gazebo_ros_control/DefaultRobotHWSim</robotSimType>
+      <legacyModeNS>true</legacyModeNS>
+    </plugin>
+  </gazebo>
 </robot>

Commit message: Update with melodic

File: sciurus17_description/urdf/sciurus17.urdf.xacro (robot description, xacro)
@@ -47,8 +47,14 @@
     </xacro:if>
     <!-- Used for fixing robot 'base_link'  to Gazebo 'world' -->
-    <link name="world"/>
-    <joint name="base_link_to_world_joint" type="fixed">
-      <parent link="world"/>
-      <child link="base_link"/>
+    <!-- <link name="world"/>                                 -->
+    <!-- <joint name="base_link_to_world_joint" type="fixed"> -->
+    <!--   <parent link="world"/>                             -->
+    <!--   <child link="base_link"/>                          -->
+    <!-- </joint>                                             -->
+    <!-- Used for fixing robot 'base_link' to Sciurus_Vehicle 'sciurus_vehicle_joint' -->
+    <link name="sciurus17_base_link"/>
+    <joint name="sciurus_vehicle_joint" type="fixed">
+      <parent link="sciurus17_base_link" />
+      <child link ="base_link" />
     </joint>
   </xacro:if>

Commit message: Fix a xacro file to use sciurus_vehicle_joint at real world

File: sciurus17_description/urdf/sciurus17.urdf.xacro (robot description, xacro)
@@ -52,11 +52,11 @@
     <!--   <child link="base_link"/>                          -->
     <!-- </joint>                                             -->
-    <!-- Used for fixing robot 'base_link' to Sciurus_Vehicle 'sciurus_vehicle_joint' -->
-    <link name="sciurus17_base_link"/>
-    <joint name="sciurus_vehicle_joint" type="fixed">
-      <parent link="sciurus17_base_link" />
-      <child link ="base_link" />
-    </joint>
   </xacro:if>
+  <!-- Used for fixing robot 'base_link' to Sciurus_Vehicle 'sciurus_vehicle_joint' -->
+  <link name="sciurus17_base_link"/>
+  <joint name="sciurus_vehicle_joint" type="fixed">
+    <parent link="sciurus17_base_link" />
+    <child link ="base_link" />
+  </joint>
   <sciurus17_body
     waist_yaw_upper_limit="${radians(-110)}"

Commit message: Add use_effort_right_arm option to xacro file

File: sciurus17_description/urdf/sciurus17.urdf.xacro (robot description, xacro)
@@ -19,14 +19,19 @@
   <xacro:arg name="load_trans2" default="false" />
   <xacro:arg name="load_trans3" default="false" />
+  <xacro:arg name="use_effort_right_arm" default="false" />
+  <xacro:property name="right_arm_interface" value="position"/>
+  <xacro:if value="$(arg use_effort_right_arm)">
+    <xacro:property name="right_arm_interface" value="effort"/>
+  </xacro:if>
   <xacro:if value="$(arg use_gazebo_simulation)">
     <xacro:include filename="$(find sciurus17_description)/urdf/sciurus17_gazebo.xacro"/>
     <xacro:if value="$(arg load_trans1)">
-      <xacro:default_transmission joint_name="r_arm_joint1"/>
-      <xacro:default_transmission joint_name="r_arm_joint2"/>
-      <xacro:default_transmission joint_name="r_arm_joint3"/>
-      <xacro:default_transmission joint_name="r_arm_joint4"/>
-      <xacro:default_transmission joint_name="r_arm_joint5"/>
-      <xacro:default_transmission joint_name="r_arm_joint6"/>
-      <xacro:default_transmission joint_name="r_arm_joint7"/>
+      <xacro:default_transmission joint_name="r_arm_joint1" interface="${right_arm_interface}"/>
+      <xacro:default_transmission joint_name="r_arm_joint2" interface="${right_arm_interface}"/>
+      <xacro:default_transmission joint_name="r_arm_joint3" interface="${right_arm_interface}"/>
+      <xacro:default_transmission joint_name="r_arm_joint4" interface="${right_arm_interface}"/>
+      <xacro:default_transmission joint_name="r_arm_joint5" interface="${right_arm_interface}"/>
+      <xacro:default_transmission joint_name="r_arm_joint6" interface="${right_arm_interface}"/>
+      <xacro:default_transmission joint_name="r_arm_joint7" interface="${right_arm_interface}"/>
       <xacro:default_transmission joint_name="r_hand_joint"/>
     </xacro:if>

File: sciurus17_description/urdf/sciurus17_gazebo.xacro (robot description, xacro)
@@ -2,5 +2,5 @@
 <robot xmlns:xacro="http://ros.org/wiki/xacro">
   <xacro:macro name="default_transmission"
-    params="joint_name">
+    params="joint_name interface:=position">
     <transmission name="${joint_name}_trans">
       <provideFeedback>true</provideFeedback>
@@ -9,8 +9,24 @@
       <type>transmission_interface/SimpleTransmission</type>
       <joint name="${joint_name}">
-        <hardwareInterface>hardware_interface/PositionJointInterface</hardwareInterface>
+        <xacro:if value="${interface == 'position'}">
+          <hardwareInterface>hardware_interface/PositionJointInterface</hardwareInterface>
+        </xacro:if>
+        <xacro:if value="${interface == 'velocity'}">
+          <hardwareInterface>hardware_interface/VelocityJointInterface</hardwareInterface>
+        </xacro:if>
+        <xacro:if value="${interface == 'effort'}">
+          <hardwareInterface>hardware_interface/EffortJointInterface</hardwareInterface>
+        </xacro:if>
       </joint>
       <actuator name="{joint_name}_motor">
-        <hardwareInterface>hardware_interface/PositionJointInterface</hardwareInterface>
+        <xacro:if value="${interface == 'position'}">
+          <hardwareInterface>hardware_interface/PositionJointInterface</hardwareInterface>
+        </xacro:if>
+        <xacro:if value="${interface == 'velocity'}">
+          <hardwareInterface>hardware_interface/VelocityJointInterface</hardwareInterface>
+        </xacro:if>
+        <xacro:if value="${interface == 'effort'}">
+          <hardwareInterface>hardware_interface/EffortJointInterface</hardwareInterface>
+        </xacro:if>
         <mechanicalReduction>1</mechanicalReduction>
       </actuator>

Commit message: Add effort control sample for left wrist

File: sciurus17_description/urdf/sciurus17.urdf.xacro (robot description, xacro)
@@ -24,4 +24,9 @@
     <xacro:property name="right_arm_interface" value="effort"/>
   </xacro:if>
+  <xacro:arg name="use_effort_left_wrist" default="false" />
+  <xacro:property name="left_wrist_interface" value="position"/>
+  <xacro:if value="$(arg use_effort_left_wrist)">
+    <xacro:property name="left_wrist_interface" value="effort"/>
+  </xacro:if>
   <xacro:if value="$(arg use_gazebo_simulation)">
     <xacro:include filename="$(find sciurus17_description)/urdf/sciurus17_gazebo.xacro"/>
@@ -43,5 +48,5 @@
       <xacro:default_transmission joint_name="l_arm_joint5"/>
       <xacro:default_transmission joint_name="l_arm_joint6"/>
-      <xacro:default_transmission joint_name="l_arm_joint7"/>
+      <xacro:default_transmission joint_name="l_arm_joint7" interface="${left_wrist_interface}"/>
       <xacro:default_transmission joint_name="l_hand_joint"/>
     </xacro:if>

Commit message: KDLはbase_linkのInertiaをサポートしていないため、実機動作時にもダミーリンク(world)を追加

File: sciurus17_description/urdf/sciurus17.urdf.xacro (robot description, xacro)
@@ -56,11 +56,11 @@
       <xacro:default_transmission joint_name="neck_pitch_joint"/>
     </xacro:if>
-    <!-- Used for fixing robot 'base_link'  to Gazebo 'world' -->
-    <link name="world"/>
-    <joint name="base_link_to_world_joint" type="fixed">
-      <parent link="world"/>
-      <child link="base_link"/>
-    </joint>
   </xacro:if>
+  <!-- Used for fixing robot 'base_link'  to Gazebo 'world' -->
+  <link name="world"/>
+  <joint name="base_link_to_world_joint" type="fixed">
+    <parent link="world"/>
+    <child link="base_link"/>
+  </joint>
   <sciurus17_body
     waist_yaw_upper_limit="${radians(-110)}"

Commit message: KDLはbase_linkのInertiaをサポートしていないため、実機動作時にもダミーリンク(world)を追加

File: sciurus17_description/urdf/sciurus17.urdf.xacro (robot description, xacro)
@@ -56,11 +56,11 @@
       <xacro:default_transmission joint_name="neck_pitch_joint"/>
     </xacro:if>
-    <!-- Used for fixing robot 'base_link'  to Gazebo 'world' -->
-    <link name="world"/>
-    <joint name="base_link_to_world_joint" type="fixed">
-      <parent link="world"/>
-      <child link="base_link"/>
-    </joint>
   </xacro:if>
+  <!-- Used for fixing robot 'base_link'  to Gazebo 'world' -->
+  <link name="world"/>
+  <joint name="base_link_to_world_joint" type="fixed">
+    <parent link="world"/>
+    <child link="base_link"/>
+  </joint>
   <xacro:sciurus17_body
     waist_yaw_upper_limit="${radians(-110)}"

Commit message: launch時のwarning消すための修正 (#122)
* KDLはbase_linkのInertiaをサポートしていないため、実機動作時にもダミーリンク(world)を追加

* kinematicsプラグインのオプションからattemptsを削除。Melodicから廃止されているため。

* KinematicsプラグインをKDLに統一

* sciurus17.srdfのtable virtual jointはスキップされているためコメントアウトする

* Add collision model to armarker link

* trac_ikを依存関係から削除

* Fix xacro file to load on Noetic environments.

* sciurus17.srdfからvirtual jointを削除。開発初期の名残で、使われていないため。

File: sciurus17_description/urdf/sciurus17.urdf.xacro (robot description, xacro)
@@ -56,12 +56,12 @@
       <xacro:default_transmission joint_name="neck_pitch_joint"/>
     </xacro:if>
-    <!-- Used for fixing robot 'base_link'  to Gazebo 'world' -->
-    <link name="world"/>
-    <joint name="base_link_to_world_joint" type="fixed">
-      <parent link="world"/>
-      <child link="base_link"/>
-    </joint>
   </xacro:if>
-  <sciurus17_body
+  <!-- Used for fixing robot 'base_link'  to Gazebo 'world' -->
+  <link name="world"/>
+  <joint name="base_link_to_world_joint" type="fixed">
+    <parent link="world"/>
+    <child link="base_link"/>
+  </joint>
+  <xacro:sciurus17_body
     waist_yaw_upper_limit="${radians(-110)}"
     waist_yaw_lower_limit="${radians(110)}"
@@ -71,6 +71,6 @@
     body_color="white"
     camera_color="white">
-  </sciurus17_body>
-  <sciurus17_head
+  </xacro:sciurus17_body>
+  <xacro:sciurus17_head
     neck_yaw_lower_limit="${radians(-165)}"
     neck_yaw_upper_limit="${radians(165)}"
@@ -81,6 +81,6 @@
     head_color="white"
     camera_color="white">
-  </sciurus17_head>
-  <sciurus17_right_arm
+  </xacro:sciurus17_head>
+  <xacro:sciurus17_right_arm
     arm_joint1_lower_limit="${radians(-90)}"
     arm_joint1_upper_limit="${radians(90)}"
@@ -100,6 +100,6 @@
     arm_joints_velocity_limit="${VELOCITY_LIMIT}"
     arm_color="white">
-  </sciurus17_right_arm>
-  <sciurus17_right_hand
+  </xacro:sciurus17_right_arm>
+  <xacro:sciurus17_right_hand
     hand_joints_lower_limit="${radians(0)}"
     hand_joints_upper_limit="${radians(86)}"
@@ -107,6 +107,6 @@
     hand_joints_velocity_limit="${VELOCITY_LIMIT}"
     hand_color="red">
-  </sciurus17_right_hand>
-  <sciurus17_left_arm
+  </xacro:sciurus17_right_hand>
+  <xacro:sciurus17_left_arm
     arm_joint1_lower_limit="${radians(-90)}"
     arm_joint1_upper_limit="${radians(90)}"
@@ -126,6 +126,6 @@
     arm_joints_velocity_limit="${VELOCITY_LIMIT}"
     arm_color="white">
-  </sciurus17_left_arm>
-  <sciurus17_left_hand
+  </xacro:sciurus17_left_arm>
+  <xacro:sciurus17_left_hand
     hand_joints_lower_limit="${radians(-86)}"
     hand_joints_upper_limit="${radians(0)}"
@@ -133,4 +133,4 @@
     hand_joints_velocity_limit="${VELOCITY_LIMIT}"
     hand_color="red">
-  </sciurus17_left_hand>
+  </xacro:sciurus17_left_hand>
 </robot>
